File: blinky.kicad_sch (KiCad schematic)
At the start: 118 parts, among them J1 Power, J3 Skedd, U1 STM32G030C6Tx, U2 BQ25570

Commit message: Sorting out DRC.
Parts:
- removed R72: 100, Resistor_SMD:R_0402_1005Metric, symbol Device:R
- removed TP1, TP2: TestPoint_Probe, Parts:TestPoint, symbol Connector:TestPoint_Probe
- added C20, C21, C22, C23, C24, C25: 100u, Capacitor_SMD:C_1206_3216Metric, symbol Device:C
- renumbered J3 to J2, R71 to R10, R73 to R18, R18 to R19, R19 to R20, R74 to R27, TP3 to TP1, TP4 to TP2, TP5 to TP3
Connections:
- net d3V3 is gone; now on net +3V3: J2.1 (Pin_1)
- net GND: now also C20.2, C21.2, C22.2, C23.2, C24.2, C25.2
- net VBatt: now also C20.1, C21.1, C22.1, C23.1, C24.1, C25.1
Other:
- moved on the sheet: C10, C11, C12, C13, C14, C15, C16, C17, C18, C19

Commit message: Cap to the max.
Parts:
- added C10, C17, C22, C29: 100u, Capacitor_SMD:C_1206_3216Metric, symbol Device:C
- added C9: 47u, Capacitor_SMD:C_0805_2012Metric, symbol Device:C
- renumbered C10 to C11, C11 to C12, C12 to C13, C13 to C14, C14 to C15, C15 to C16, C16 to C18, C17 to C19, C18 to C20, C19 to C21, C20 to C23, C21 to C24, C22 to C25, C23 to C26, C24 to C27, C25 to C28
Connections:
- net +3V3: no longer U1.4 (VBAT)
- net GND: now also C10.2, C17.2, C22.2, C29.2, C9.1
- net VBatt: now also C10.1, C17.1, C22.1, C29.1
- new net: C9.2, U1.4 (VBAT)
Other:
- moved on the sheet: C11, C12, C13, C14, C15, C16, C18, C19, C20, C21, C23, C24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

Commit message: Sort out resistor values.
Parts:
- R1: value 634k -> 1M8
- R10, R27: value 100k -> 10k; LCSC C25741 -> C25744
- R11, R12, R13, R14, R15, R16, R21, R22, R23, R24, R25, R26, R31, R32, R33, R34, R35, R36, R41, R42, R43, R44, R45, R46, R51, R52, R53, R54, R55, R56, R61, R62, R63, R64, R65, R66: value 100 -> 470; LCSC C25076 -> C25117
- R2: value 6M2 -> 6M8
- R3: value 3M9 -> 2M2; LCSC (none) -> C22938
- R4: value 5M1 -> 6M2
- R5: value 430k -> 330k; LCSC C23203 -> C23137
- R6: value 3M9 -> 3M; LCSC (none) -> C23156
- R7: value 6M8 -> 5M1; LCSC (none) -> C13320
- R8: value 330k -> 750k; LCSC C23137 -> C23240
- R9: value 3M6 -> 2M2; LCSC (none) -> C22938
Other:
- note added: "3.3V, 4.95V"
- note added: "5.1V"
- note removed: "2.86V, 3.13V"
- note removed: "3.95V"

Commit message: Flip debug connector.
Parts:
- R3, R6, R7, R9: now in the parts list
Changed lines of the file:
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@@
 		(unit 1)
 		(exclude_from_sim no)
-		(in_bom no)
+		(in_bom yes)
 		(on_board yes)
 		(dnp no)
@@
 		(unit 1)
 		(exclude_from_sim no)
-		(in_bom no)
+		(in_bom yes)
 		(on_board yes)
 		(dnp no)
@@
 		(unit 1)
 		(exclude_from_sim no)
-		(in_bom no)
+		(in_bom yes)
 		(on_board yes)
 		(dnp no)
@@
 		(unit 1)
 		(exclude_from_sim no)
-		(in_bom no)
+		(in_bom yes)
 		(on_board yes)
 		(dnp no)

Commit message: Use 330 ohm resistors.
Parts:
- L1, L2: now in the parts list
- R11, R12, R13, R14, R15, R16, R21, R22, R23, R24, R25, R26, R31, R32, R33, R34, R35, R36, R41, R42, R43, R44, R45, R46, R51, R52, R53, R54, R55, R56, R61, R62, R63, R64, R65, R66: value 470 -> 330; LCSC C25117 -> C25104

Commit message: Believe the datasheet not the website
Parts:
- added C30: 10u, Capacitor_SMD:C_0603_1608Metric, symbol Device:C
- L1, L2: footprint Inductor_SMD:L_0805_2012Metric_Pad1.05x1.20mm_HandSolder -> Parts:L_1008_2520Metric-Adjusted
Connections:
- net GND: now also C30.2
- net VBatt: now also C30.1
Changed lines of the file:
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@@
 	)
 	(junction
-		(at 97.79 38.1)
-		(diameter 0)
-		(color 0 0 0 0)
-	)
-	(junction
 		(at 185.42 109.22)
 		(diameter 0)
@@
 	)
 	(junction
+		(at 100.33 38.1)
+		(diameter 0)
+		(color 0 0 0 0)
+	)
+	(junction
 		(at 215.9 48.26)
 		(diameter 0)
@@
 	(wire
 		(pts
-			(xy 90.17 38.1) (xy 97.79 38.1)
+			(xy 90.17 38.1) (xy 100.33 38.1)
 		)
 		(stroke
@@
 	(wire
 		(pts
+			(xy 100.33 38.1) (xy 101.6 38.1)
+		)
+		(stroke
+			(width 0)
+			(type default)
+		)
+	)
+	(wire
+		(pts
 			(xy 238.76 109.22) (xy 246.38 109.22)
 		)
@@
 	(wire
 		(pts
+			(xy 109.22 38.1) (xy 110.49 38.1)
+		)
+		(stroke
+			(width 0)
+			(type default)
+		)
+	)
+	(wire
+		(pts
 			(xy 200.66 48.26) (xy 205.74 48.26)
 		)
@@
 	(wire
 		(pts
-			(xy 97.79 38.1) (xy 105.41 38.1)
-		)
-		(stroke
-			(width 0)
-			(type default)
-		)
-	)
-	(wire
-		(pts
 			(xy 104.14 151.13) (xy 111.76 151.13)
 		)
@@
 	)
 	(label "VBatt"
-		(at 105.41 38.1 180)
+		(at 99.06 38.1 180)
 		(effects
 			(font
@@
 	(symbol
 		(lib_id "power:PWR_FLAG")
-		(at 97.79 38.1 0)
+		(at 100.33 38.1 0)
 		(mirror y)
 		(unit 1)
@@
 		(dnp no)
 		(property "Reference" "#FLG03"
-			(at 97.79 36.195 0)
+			(at 100.33 36.195 0)
 			(effects
 				(font
@@
 		)
 		(property "Value" "PWR_FLAG"
-			(at 97.79 34.29 0)
+			(at 100.33 34.29 0)
 			(effects
 				(font
@@
 		)
 		(property "Footprint" ""
-			(at 97.79 38.1 0)
+			(at 100.33 38.1 0)
 			(effects
 				(font
@@
 		)
 		(property "Datasheet" "~"
-			(at 97.79 38.1 0)
+			(at 100.33 38.1 0)
 			(effects
 				(font
@@
 		)
 		(property "Description" "Special symbol for telling ERC where power comes from"
-			(at 97.79 38.1 0)
+			(at 100.33 38.1 0)
 			(effects
 				(font
@@
 	)
 	(symbol
+		(lib_id "Device:C")
+		(at 105.41 38.1 90)
+		(unit 1)
+		(exclude_from_sim no)
+		(in_bom yes)
+		(on_board yes)
+		(dnp no)
+		(property "Reference" "C30"
+			(at 105.41 35.56 90)
+			(effects
+				(font
+					(size 1.27 1.27)
+				)
+				(justify top)
+			)
+		)
+		(property "Value" "10u"
+			(at 106.426 37.846 90)
+			(effects
+				(font
+					(size 1.27 1.27)
+				)
+				(justify right top)
+			)
+		)
+		(property "Footprint" "Capacitor_SMD:C_0603_1608Metric"
+			(at 109.22 37.1348 0)
+			(effects
+				(font
+					(size 1.27 1.27)
+				)
+				(hide yes)
+			)
+		)
+		(property "Datasheet" "~"
+			(at 105.41 38.1 0)
+			(effects
+				(font
+					(size 1.27 1.27)
+				)
+				(hide yes)
+			)
+		)
+		(property "Description" "Unpolarized capacitor"
+			(at 105.41 38.1 0)
+			(effects
+				(font
+					(size 1.27 1.27)
+				)
+				(hide yes)
+			)
+		)
+		(property "LCSC" "C19702"
+			(at 105.41 38.1 0)
+			(effects
+				(font
+					(size 1.27 1.27)
+				)
+				(hide yes)
+			)
+		)
+		(pin "2"
+		)
+		(pin "1"
+		)
+		(instances
+			(project "blinky"
+				(path "/78e97d1e-72bf-4146-b73c-dacf670385a3"
+					(reference "C30")
+					(unit 1)
+				)
+			)
+		)
+	)
+	(symbol
 		(lib_id "Device:LED")
 		(at 231.14 143.51 90)
@@
 			)
 		)
-		(property "Footprint" "Inductor_SMD:L_0805_2012Metric_Pad1.05x1.20mm_HandSolder"
+		(property "Footprint" "Parts:L_1008_2520Metric-Adjusted"
 			(at 66.04 45.72 0)
 			(effects
@@
 	)
 	(symbol
+		(lib_id "power:GND")
+		(at 110.49 38.1 0)
+		(unit 1)
+		(exclude_from_sim no)
+		(in_bom yes)
+		(on_board yes)
+		(dnp no)
+		(property "Reference" "#PWR026"
+			(at 110.49 44.45 0)
+			(effects
+				(font
+					(size 1.27 1.27)
+				)
+				(hide yes)
+			)
+		)
+		(property "Value" "GND"
+			(at 110.49 41.91 0)
+			(effects
+				(font
+					(size 1.27 1.27)
+				)
+			)
+		)
+		(property "Footprint" ""
+			(at 110.49 38.1 0)
+			(effects
+				(font
+					(size 1.27 1.27)
+				)
+				(hide yes)
+			)
+		)
+		(property "Datasheet" ""
+			(at 110.49 38.1 0)
+			(effects
+				(font
+					(size 1.27 1.27)
+				)
+				(hide yes)
+			)
+		)
+		(property "Description" "Power symbol creates a global label with name \"GND\" , ground"
+			(at 110.49 38.1 0)
+			(effects
+				(font
+					(size 1.27 1.27)
+				)
+				(hide yes)
+			)
+		)
+		(pin "1"
+		)
+		(instances
+			(project "blinky"
+				(path "/78e97d1e-72bf-4146-b73c-dacf670385a3"
+					(reference "#PWR026")
+					(unit 1)
+				)
+			)
+		)
+	)
+	(symbol
 		(lib_id "Device:R")
 		(at 147.32 67.31 90)
@@
 			)
 		)
-		(property "Footprint" "Inductor_SMD:L_0805_2012Metric_Pad1.05x1.20mm_HandSolder"
+		(property "Footprint" "Parts:L_1008_2520Metric-Adjusted"
 			(at 107.95 45.72 0)
 			(effects

Commit message: Some more animations.
Parts:
- R1: value 1M8 -> 2M7
- R2: value 6M8 -> 1M8
Other:
- note added: "2.2V to 3.xV"
- note removed: "3.3V, 4.95V"
Changed lines of the file:
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@@
 		)
 	)
-	(text "3.3V, 4.95V"
+	(text "2.2V to 3.xV"
 		(exclude_from_sim no)
 		(at 140.97 50.8 0)
@@
 	)
 	(junction
+		(at 135.89 60.96)
+		(diameter 0)
+		(color 0 0 0 0)
+	)
+	(junction
 		(at 195.58 48.26)
 		(diameter 0)
@@
 	)
 	(junction
-		(at 135.89 60.96)
-		(diameter 0)
-		(color 0 0 0 0)
-	)
-	(junction
 		(at 190.5 57.15)
 		(diameter 0)
@@
 	)
 	(junction
+		(at 128.27 60.96)
+		(diameter 0)
+		(color 0 0 0 0)
+	)
+	(junction
 		(at 208.28 78.74)
 		(diameter 0)
@@
 	)
 	(junction
-		(at 128.27 60.96)
-		(diameter 0)
-		(color 0 0 0 0)
-	)
-	(junction
 		(at 190.5 40.64)
 		(diameter 0)
@@
 	(wire
 		(pts
-			(xy 128.27 60.96) (xy 128.27 67.31)
+			(xy 170.18 147.32) (xy 170.18 149.86)
 		)
 		(stroke
@@
 	(wire
 		(pts
-			(xy 170.18 147.32) (xy 170.18 149.86)
+			(xy 177.8 109.22) (xy 185.42 109.22)
 		)
 		(stroke
@@
 	(wire
 		(pts
-			(xy 177.8 109.22) (xy 185.42 109.22)
+			(xy 128.27 53.34) (xy 128.27 60.96)
 		)
 		(stroke
@@
 	(wire
 		(pts
-			(xy 128.27 53.34) (xy 128.27 60.96)
-		)
-		(stroke
-			(width 0)
-			(type default)
-		)
-	)
-	(wire
-		(pts
 			(xy 177.8 86.36) (xy 177.8 88.9)
 		)
@@
 	(wire
 		(pts
+			(xy 128.27 60.96) (xy 128.27 67.31)
+		)
+		(stroke
+			(width 0)
+			(type default)
+		)
+	)
+	(wire
+		(pts
 			(xy 200.66 57.15) (xy 195.58 57.15)
 		)
@@
 			)
 		)
-		(property "Value" "1M8"
+		(property "Value" "2M7"
 			(at 132.08 53.34 90)
 			(effects
@@
 		(dnp no)
 		(property "Reference" "R3"
-			(at 147.32 54.864 90)
+			(at 147.32 54.61 90)
 			(effects
 				(font
@@
 		(dnp no)
 		(property "Reference" "R6"
-			(at 147.32 62.484 90)
+			(at 147.32 62.23 90)
 			(effects
 				(font
@@
 			)
 		)
-		(property "Value" "6M8"
+		(property "Value" "1M8"
 			(at 139.7 53.34 90)
 			(effects
@@
 		(dnp no)
 		(property "Reference" "R9"
-			(at 147.32 68.834 90)
+			(at 147.32 68.58 90)
 			(effects
 				(font
